Commit message: Finished making small robot and etc

File: urdf/gillwald_bot_small/gillwald_bot_small.xacro (robot description, xacro)
@@ -9,5 +9,5 @@
     <inertial>
       <mass value="5"/>
-      <origin rpy="0 0 0" xyz="0 0 0.1"/>
+      <origin rpy="0 0 0" xyz="0 0 0"/>
       <inertia ixx="0.0395416666667" ixy="0" ixz="0" iyy="0.106208333333" iyz="0" izz="0.106208333333"/>
     </inertial>
@@ -15,5 +15,5 @@
     <collision name="collision_chassis">
       <geometry>
-        <box size="0.5 0.3 0.1"/>
+        <box size="0.2032 0.13335 0.1016"/>
       </geometry>
     </collision>
@@ -21,5 +21,5 @@
       <origin rpy="0 0 0" xyz="0 0 0"/>
       <geometry>
-        <box size="0.5 0.3 0.1"/>
+        <box size="0.2032 0.13335 0.1016"/>
       </geometry>
       <material name="blue"/>
@@ -27,7 +27,7 @@
     <!-- caster front -->
     <collision name="caster_front_collision">
-      <origin rpy=" 0 0 0" xyz="0.2 0 -0.05"/>
+      <origin rpy=" 0 0 0" xyz="0.0762 0 -0.0508"/>
       <geometry>
-        <sphere radius="0.05"/>
+        <sphere radius="0.0127"/>
       </geometry>
       <surface>
@@ -43,7 +43,7 @@
     </collision>
     <visual name="caster_front_visual">
-      <origin rpy=" 0 0 0" xyz="0.2 0 -0.05"/>
+      <origin rpy=" 0 0 0" xyz="0.0762 0 -0.0508"/>
       <geometry>
-        <sphere radius="0.05"/>
+        <sphere radius="0.0127"/>
       </geometry>
     </visual>
@@ -51,30 +51,30 @@
   <link name="sensor_laser">
     <inertial>
-      <origin xyz="0 0 -0.025" rpy="0 0 0" />
+      <origin xyz="0 0 0" rpy="0 0 0" />
       <mass value="1" />
-      <xacro:cylinder_inertia mass="1" r="0.05" l="0.1" />
+      <xacro:cylinder_inertia mass="0.5" r="0.0381" l="0.0508" />
     </inertial>
     <visual>
-      <origin xyz="0 0 -0.025" rpy="0 0 0" />
+      <origin xyz="0 0 0" rpy="0 0 0" />
       <geometry>
-        <cylinder radius="0.05" length="0.1"/>
+        <cylinder radius="0.0381" length="0.0508"/>
       </geometry>
       <material name="white" />
     </visual>
     <collision>
-      <origin xyz="0 0 -0.025" rpy="0 0 0"/>
+      <origin xyz="0 0 0" rpy="0 0 0"/>
       <geometry>
-        <cylinder radius="0.05" length="0.1"/>
+        <cylinder radius="0.0381" length="0.0508"/>
       </geometry>
     </collision>
   </link>
   <joint name="joint_sensor_laser" type="fixed">
-    <origin xyz="0.15 0 0.125" rpy="0 0 0"/>
+    <origin xyz="0.0508 0 0.0762" rpy="0 0 0"/>
     <parent link="link_chassis"/>
     <child link="sensor_laser"/>
   </joint>
   <xacro:link_wheel name="link_right_wheel" />
-  <xacro:joint_wheel name="joint_right_wheel" child="link_right_wheel" origin_xyz="-0.15 0.20 0" />
+  <xacro:joint_wheel name="joint_right_wheel" child="link_right_wheel" origin_xyz="-0.0762 0.079375 -0.0254" />
   <xacro:link_wheel name="link_left_wheel" />
-  <xacro:joint_wheel name="joint_left_wheel" child="link_left_wheel" origin_xyz="-0.15 -0.20 0" />
+  <xacro:joint_wheel name="joint_left_wheel" child="link_left_wheel" origin_xyz="-0.0762 -0.079375 -0.0254" />
 </robot>

File: urdf/gillwald_bot_small/macros_small.xacro (robot description, xacro)
@@ -11,5 +11,5 @@
               <origin rpy="0 1.5707 1.5707" xyz="0 0 0"/>
               <geometry>
-                <cylinder length="0.04" radius="0.1"/>
+                <cylinder length="0.0254" radius="0.0381"/>
               </geometry>
             </collision>
@@ -17,5 +17,5 @@
               <origin rpy="0 1.5707 1.5707" xyz="0 0 0"/>
               <geometry>
-                <cylinder length="0.04" radius="0.1"/>
+                <cylinder length="0.0254" radius="0.0381"/>
               </geometry>
             </visual>
